File: RC-Substitution-Box.kicad_pcb (KiCad board)
At the start: 2 copper layers, 103 x 85 mm, 64 parts, among them J13 Screw_Terminal_01x02, J14 Screw_Terminal_01x02, J5 Screw_Terminal_01x02, J6 Screw_Terminal_01x02, SW2 208-12, SW3 208-12, SW4 208-12, SW5 100SP3T1B1M2QE-ND, SW6 208-12, SW7 100SP3T1B1M2QE-ND

Commit message: Removing SW and adding Axial RC Option
-Removing the SW becasue it is not needed
- Adding an axial option just for flexibility
Parts:
- added C25: 100p, Capacitor_THT:C_Disc_D5.1mm_W3.2mm_P5.00mm, F.Cu at (343.2, 83.0)
- added C26: 200p, Capacitor_THT:C_Disc_D5.1mm_W3.2mm_P5.00mm, F.Cu at (343.2, 87.7)
- added C27: 400p, Capacitor_THT:C_Disc_D5.1mm_W3.2mm_P5.00mm, F.Cu at (343.2, 92.5)
- added C28: 800p, Capacitor_THT:C_Disc_D5.1mm_W3.2mm_P5.00mm, F.Cu at (343.2, 97.2)
- added C29: 1u, Capacitor_THT:C_Disc_D5.1mm_W3.2mm_P5.00mm, F.Cu at (351.3, 83.0)
- added C30: 2u, Capacitor_THT:C_Disc_D5.1mm_W3.2mm_P5.00mm, F.Cu at (351.3, 87.7)
- added C31: 4u, Capacitor_THT:C_Disc_D5.1mm_W3.2mm_P5.00mm, F.Cu at (351.3, 92.5)
- added C32: 8u, Capacitor_THT:C_Disc_D5.1mm_W3.2mm_P5.00mm, F.Cu at (351.3, 97.2)
- added C33: 16u, Capacitor_THT:C_Disc_D5.1mm_W3.2mm_P5.00mm, F.Cu at (359.5, 83.0)
- added C34: 32u, Capacitor_THT:C_Disc_D5.1mm_W3.2mm_P5.00mm, F.Cu at (359.5, 87.7)
- added C35: 64u, Capacitor_THT:C_Disc_D5.1mm_W3.2mm_P5.00mm, F.Cu at (359.5, 92.5)
- added C36: 128u, Capacitor_THT:C_Disc_D5.1mm_W3.2mm_P5.00mm, F.Cu at (359.5, 97.2)
- added J15: Screw_Terminal_01x02, TerminalBlock_Phoenix:TerminalBlock_Phoenix_MKDS-1,5-2_1x02_P5.00mm_Horizontal, F.Cu at (346.4, 74.7)
- added J7: Screw_Terminal_01x02, TerminalBlock_Phoenix:TerminalBlock_Phoenix_MKDS-1,5-2_1x02_P5.00mm_Horizontal, F.Cu at (322.3, 74.7)
- added R22: 0-100, DJ-FOOTPRINTS:RES-ADJ-TH_3P-L9.5-W9.5-P2.54-BR-BS, F.Cu at (346.9, 105.0)
- added R39: 100, Resistor_THT:R_Axial_DIN0207_L6.3mm_D2.5mm_P7.62mm_Horizontal, F.Cu at (309.6, 70.5)
- added R40: 200, Resistor_THT:R_Axial_DIN0207_L6.3mm_D2.5mm_P7.62mm_Horizontal, F.Cu at (309.6, 74.6)
- added R41: 400, Resistor_THT:R_Axial_DIN0207_L6.3mm_D2.5mm_P7.62mm_Horizontal, F.Cu at (309.6, 78.6)
- added R42: 800, Resistor_THT:R_Axial_DIN0207_L6.3mm_D2.5mm_P7.62mm_Horizontal, F.Cu at (309.6, 82.7)
- added R43: 1K6, Resistor_THT:R_Axial_DIN0207_L6.3mm_D2.5mm_P7.62mm_Horizontal, F.Cu at (309.6, 86.7)
- added R44: 3K2, Resistor_THT:R_Axial_DIN0207_L6.3mm_D2.5mm_P7.62mm_Horizontal, F.Cu at (309.6, 90.8)
- added R45: 6K4, Resistor_THT:R_Axial_DIN0207_L6.3mm_D2.5mm_P7.62mm_Horizontal, F.Cu at (309.6, 94.8)
- added R46: 12K8, Resistor_THT:R_Axial_DIN0207_L6.3mm_D2.5mm_P7.62mm_Horizontal, F.Cu at (309.6, 98.9)
- added R47: 25K6, Resistor_THT:R_Axial_DIN0207_L6.3mm_D2.5mm_P7.62mm_Horizontal, F.Cu at (309.6, 102.9)
- added R48: 51K2, Resistor_THT:R_Axial_DIN0207_L6.3mm_D2.5mm_P7.62mm_Horizontal, F.Cu at (309.6, 107.0)
- added R49: 102K4, Resistor_THT:R_Axial_DIN0207_L6.3mm_D2.5mm_P7.62mm_Horizontal, F.Cu at (309.6, 111.0)
- added R50: 204K2, Resistor_THT:R_Axial_DIN0207_L6.3mm_D2.5mm_P7.62mm_Horizontal, F.Cu at (309.6, 115.1)
- SW5, SW7: value 100SP3T1B1M2QE-ND -> 208-12; footprint DJ-FOOTPRINTS:SW_100SP3T1B1M2QE -> Button_Switch_THT:SW_DIP_SPSTx12_Slide_9.78x32.66mm_W7.62mm_P2.54mm
- moved SW7 211.6 mm to (332.1, 83.8), turned to 0 degrees
- moved SW5 154.8 mm to (297.4, 72.3), turned to 0 degrees
- moved G*** 94.8 mm to (53.5, 101.0)
- moved H4 42.5 mm to (140.2, 145.7)
- moved H3 41.7 mm to (220.5, 47.5)
- moved R22 41.2 mm to (78.7, 105.2)
- moved H2 40.3 mm to (51.7, 124.2)
- moved J13 31.3 mm to (139.0, 115.5), turned to 180 degrees
- moved C13 20.0 mm to (161.4, 63.2)
- moved C14 20.0 mm to (161.4, 65.5)
- moved C15 20.0 mm to (161.4, 67.9)
- moved C16 20.0 mm to (161.4, 70.2)
- moved C17 20.0 mm to (161.4, 72.6)
- moved C18 20.0 mm to (161.4, 74.9)
- moved C19 20.0 mm to (161.4, 77.3)
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Connections:
- J5 pad 2: Net-(J13-Pin_2) -> Net-(J5-Pin_2)
- J6 pad 2: Net-(J14-Pin_2) -> Net-(J6-Pin_2)
- SW2 pad 1: Net-(J14-Pin_2) -> Net-(J6-Pin_2)
- SW2 pad 10: Net-(J14-Pin_2) -> Net-(J6-Pin_2)
- SW2 pad 11: Net-(J14-Pin_2) -> Net-(J6-Pin_2)
- SW2 pad 12: Net-(J14-Pin_2) -> Net-(J6-Pin_2)
- SW2 pad 2: Net-(J14-Pin_2) -> Net-(J6-Pin_2)
- SW2 pad 3: Net-(J14-Pin_2) -> Net-(J6-Pin_2)
- SW2 pad 4: Net-(J14-Pin_2) -> Net-(J6-Pin_2)
- SW2 pad 5: Net-(J14-Pin_2) -> Net-(J6-Pin_2)
- SW2 pad 6: Net-(J14-Pin_2) -> Net-(J6-Pin_2)
- SW2 pad 7: Net-(J14-Pin_2) -> Net-(J6-Pin_2)
- SW2 pad 8: Net-(J14-Pin_2) -> Net-(J6-Pin_2)
- SW2 pad 9: Net-(J14-Pin_2) -> Net-(J6-Pin_2)
- SW4 pad 1: Net-(J13-Pin_2) -> Net-(J5-Pin_2)
- SW4 pad 10: Net-(J13-Pin_2) -> Net-(J5-Pin_2)
- SW4 pad 11: Net-(J13-Pin_2) -> Net-(J5-Pin_2)
- SW4 pad 12: Net-(J13-Pin_2) -> Net-(J5-Pin_2)
- SW4 pad 2: Net-(J13-Pin_2) -> Net-(J5-Pin_2)
- SW4 pad 3: Net-(J13-Pin_2) -> Net-(J5-Pin_2)
- SW4 pad 4: Net-(J13-Pin_2) -> Net-(J5-Pin_2)
- SW4 pad 5: Net-(J13-Pin_2) -> Net-(J5-Pin_2)
- SW4 pad 6: Net-(J13-Pin_2) -> Net-(J5-Pin_2)
- SW4 pad 7: Net-(J13-Pin_2) -> Net-(J5-Pin_2)
- SW4 pad 8: Net-(J13-Pin_2) -> Net-(J5-Pin_2)
- SW4 pad 9: Net-(J13-Pin_2) -> Net-(J5-Pin_2)
- SW5 pad 1: Net-(J5-Pin_1) -> Net-(R39-Pad2)
- SW5 pad 2: Net-(J13-Pin_1) -> Net-(R40-Pad2)
- SW5 pad 3: Net-(J13-Pin_2) -> Net-(R41-Pad2)
- SW7 pad 1: Net-(J6-Pin_1) -> Net-(J7-Pin_2)
- SW7 pad 2: Net-(J14-Pin_1) -> Net-(J7-Pin_2)
- SW7 pad 3: Net-(J14-Pin_2) -> Net-(J7-Pin_2)
Routing:
- net Net-(J13-Pin_2): track 122.7 -> 4.54 mm
- net Net-(J14-Pin_2): track 96.2 -> 0.00 mm
- net Net-(J6-Pin_1): track 98.5 -> 30.3 mm
- net Net-(R22-Pad1): track 86.4 -> 25.8 mm
- net Net-(J13-Pin_1): track 65.3 -> 17.4 mm
- net Net-(J5-Pin_1): track 71.7 -> 27.1 mm
- net Net-(J14-Pin_1): track 47.9 -> 7.91 mm
- net Net-(J6-Pin_2): track 0.00 -> 27.9 mm
- net Net-(J5-Pin_2): track 0.00 -> 27.9 mm
Other:
- board outline removed
- board text removed: "Parallel RC"
- board text removed: "R"
- board text removed: "Series RC"

Commit message: updated layout
Parts:
- removed R22 (x2): 0-100, DJ-FOOTPRINTS:RES-ADJ-TH_3P-L9.5-W9.5-P2.54-BR-BS
- added JP1: SolderJumper_2_Open, Jumper:SolderJumper-2_P1.3mm_Open_Pad1.0x1.5mm, F.Cu at (87.0, 96.0)
- added RPONT: 0-100, DJ-FOOTPRINTS:RES-ADJ-TH_3P-L9.5-W9.5-P2.54-BR-BS, F.Cu at (80.0, 96.0)
- moved J15 186.3 mm to (163.1, 108.6)
- moved C33 157.5 mm to (202.0, 84.5)
- moved C34 157.5 mm to (202.0, 88.5)
- moved C36 157.5 mm to (202.0, 96.5)
- moved C35 157.5 mm to (202.0, 92.5)
- moved C32 150.3 mm to (202.0, 80.5)
- moved C31 150.2 mm to (202.0, 76.5)
- moved C30 150.1 mm to (202.0, 72.5)
- moved C29 150.0 mm to (202.0, 68.5)
- moved C28 144.9 mm to (202.0, 64.5)
- moved SW7 144.8 mm to (189.9, 57.0)
- moved C27 144.8 mm to (202.0, 60.5)
- moved C26 144.6 mm to (202.0, 56.5)
- moved C25 144.4 mm to (202.0, 52.5)
- moved R44 138.3 mm to (174.4, 61.6), turned to -90 degrees
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Connections:
- C1 pad 2: Net-(J6-Pin_1) -> Net-(J6-Pin_2)
- C10 pad 2: Net-(J6-Pin_1) -> Net-(J6-Pin_2)
- C11 pad 2: Net-(J6-Pin_1) -> Net-(J6-Pin_2)
- C12 pad 2: Net-(J6-Pin_1) -> Net-(J6-Pin_2)
- C13 pad 2: Net-(J5-Pin_1) -> Net-(J5-Pin_2)
- C14 pad 2: Net-(J5-Pin_1) -> Net-(J5-Pin_2)
- C15 pad 2: Net-(J5-Pin_1) -> Net-(J5-Pin_2)
- C16 pad 2: Net-(J5-Pin_1) -> Net-(J5-Pin_2)
- C17 pad 2: Net-(J5-Pin_1) -> Net-(J5-Pin_2)
- C18 pad 2: Net-(J5-Pin_1) -> Net-(J5-Pin_2)
- C19 pad 2: Net-(J5-Pin_1) -> Net-(J5-Pin_2)
- C2 pad 2: Net-(J6-Pin_1) -> Net-(J6-Pin_2)
- C20 pad 2: Net-(J5-Pin_1) -> Net-(J5-Pin_2)
- C21 pad 2: Net-(J5-Pin_1) -> Net-(J5-Pin_2)
- C22 pad 2: Net-(J5-Pin_1) -> Net-(J5-Pin_2)
- C23 pad 2: Net-(J5-Pin_1) -> Net-(J5-Pin_2)
- C24 pad 2: Net-(J5-Pin_1) -> Net-(J5-Pin_2)
- C25 pad 2: Net-(J7-Pin_1) -> Net-(J7-Pin_2)
- C26 pad 2: Net-(J7-Pin_1) -> Net-(J7-Pin_2)
- C27 pad 2: Net-(J7-Pin_1) -> Net-(J7-Pin_2)
- C28 pad 2: Net-(J7-Pin_1) -> Net-(J7-Pin_2)
- C29 pad 2: Net-(J7-Pin_1) -> Net-(J7-Pin_2)
- C3 pad 2: Net-(J6-Pin_1) -> Net-(J6-Pin_2)
- C30 pad 2: Net-(J7-Pin_1) -> Net-(J7-Pin_2)
- C31 pad 2: Net-(J7-Pin_1) -> Net-(J7-Pin_2)
- C32 pad 2: Net-(J7-Pin_1) -> Net-(J7-Pin_2)
- C33 pad 2: Net-(J7-Pin_1) -> Net-(J7-Pin_2)
- C34 pad 2: Net-(J7-Pin_1) -> Net-(J7-Pin_2)
- C35 pad 2: Net-(J7-Pin_1) -> Net-(J7-Pin_2)
- C36 pad 2: Net-(J7-Pin_1) -> Net-(J7-Pin_2)
- C4 pad 2: Net-(J6-Pin_1) -> Net-(J6-Pin_2)
- C5 pad 2: Net-(J6-Pin_1) -> Net-(J6-Pin_2)
- C6 pad 2: Net-(J6-Pin_1) -> Net-(J6-Pin_2)
- C7 pad 2: Net-(J6-Pin_1) -> Net-(J6-Pin_2)
- C8 pad 2: Net-(J6-Pin_1) -> Net-(J6-Pin_2)
- C9 pad 2: Net-(J6-Pin_1) -> Net-(J6-Pin_2)
- SW2 pad 1: Net-(J6-Pin_2) -> Net-(J6-Pin_1)
- SW2 pad 10: Net-(J6-Pin_2) -> Net-(J6-Pin_1)
- SW2 pad 11: Net-(J6-Pin_2) -> Net-(J6-Pin_1)
- SW2 pad 12: Net-(J6-Pin_2) -> Net-(J6-Pin_1)
- SW2 pad 2: Net-(J6-Pin_2) -> Net-(J6-Pin_1)
- SW2 pad 3: Net-(J6-Pin_2) -> Net-(J6-Pin_1)
- SW2 pad 4: Net-(J6-Pin_2) -> Net-(J6-Pin_1)
- SW2 pad 5: Net-(J6-Pin_2) -> Net-(J6-Pin_1)
- SW2 pad 6: Net-(J6-Pin_2) -> Net-(J6-Pin_1)
- SW2 pad 7: Net-(J6-Pin_2) -> Net-(J6-Pin_1)
- SW2 pad 8: Net-(J6-Pin_2) -> Net-(J6-Pin_1)
- SW2 pad 9: Net-(J6-Pin_2) -> Net-(J6-Pin_1)
- SW4 pad 1: Net-(J5-Pin_2) -> Net-(J5-Pin_1)
- SW4 pad 10: Net-(J5-Pin_2) -> Net-(J5-Pin_1)
- SW4 pad 11: Net-(J5-Pin_2) -> Net-(J5-Pin_1)
- SW4 pad 12: Net-(J5-Pin_2) -> Net-(J5-Pin_1)
- SW4 pad 2: Net-(J5-Pin_2) -> Net-(J5-Pin_1)
- SW4 pad 3: Net-(J5-Pin_2) -> Net-(J5-Pin_1)
- SW4 pad 4: Net-(J5-Pin_2) -> Net-(J5-Pin_1)
- SW4 pad 5: Net-(J5-Pin_2) -> Net-(J5-Pin_1)
- SW4 pad 6: Net-(J5-Pin_2) -> Net-(J5-Pin_1)
- SW4 pad 7: Net-(J5-Pin_2) -> Net-(J5-Pin_1)
- SW4 pad 8: Net-(J5-Pin_2) -> Net-(J5-Pin_1)
- SW4 pad 9: Net-(J5-Pin_2) -> Net-(J5-Pin_1)
- SW7 pad 1: Net-(J7-Pin_2) -> Net-(J7-Pin_1)
- SW7 pad 10: Net-(J7-Pin_2) -> Net-(J7-Pin_1)
- SW7 pad 11: Net-(J7-Pin_2) -> Net-(J7-Pin_1)
- SW7 pad 12: Net-(J7-Pin_2) -> Net-(J7-Pin_1)
- SW7 pad 2: Net-(J7-Pin_2) -> Net-(J7-Pin_1)
- SW7 pad 3: Net-(J7-Pin_2) -> Net-(J7-Pin_1)
- SW7 pad 4: Net-(J7-Pin_2) -> Net-(J7-Pin_1)
- SW7 pad 5: Net-(J7-Pin_2) -> Net-(J7-Pin_1)
- SW7 pad 6: Net-(J7-Pin_2) -> Net-(J7-Pin_1)
- SW7 pad 7: Net-(J7-Pin_2) -> Net-(J7-Pin_1)
- SW7 pad 8: Net-(J7-Pin_2) -> Net-(J7-Pin_1)
- SW7 pad 9: Net-(J7-Pin_2) -> Net-(J7-Pin_1)
Routing:
- net Net-(J13-Pin_2): track 4.54 -> 62.9 mm
- net Net-(JP1-B): track 25.8 -> 80.9 mm
- net Net-(J7-Pin_1): track 0.00 -> 52.1 mm
- net Net-(J14-Pin_1): track 7.91 -> 39.0 mm
- net Net-(J6-Pin_2): track 27.9 -> 53.9 mm
- net Net-(J5-Pin_2): track 27.9 -> 53.7 mm
- net Net-(J5-Pin_1): track 27.1 -> 52.2 mm
- net Net-(J14-Pin_2): track 0.00 -> 24.5 mm
- net Net-(J15-Pin_1): track 0.00 -> 24.2 mm
- net Net-(R39-Pad2): track 0.00 -> 23.0 mm
- net Net-(J6-Pin_1): track 30.3 -> 52.1 mm
- net Net-(J13-Pin_1): track 17.4 -> 38.0 mm
- net Net-(R40-Pad2): track 0.00 -> 17.7 mm
- net Net-(C36-Pad1): track 0.00 -> 13.5 mm
- net Net-(C35-Pad1): track 0.00 -> 12.0 mm
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Other:
- board outline added: 146.5 x 75.5 mm
- board text added: "AXIAL RC SUBSTITUTION"
- board text added: "Capacitor Axial"
- board text added: "Capacitor General"
- board text added: "Capacitor Precision"
- board text added: "Fine Tune Potentiometer"
- board text added: "GENERAL RC SUBSTITUTION"
- board text added: "Main Sheet"
- board text added: "PRECISION RC SUBSTITUTION"
- board text added: "Potentiometer Bypass"
- board text added: "REV.A Made by DJ"
- board text added: "Resistor Axial"
- board text added: "Resistor General"
- board text added: "Resistor Precision"
- board text removed: "BINARY GENERAL RC SUBSTITUTION"
- board text removed: "BINARY PRECISION RC SUBSTITUTION"
- board text removed: "Capacitor & Series RC"
- board text removed: "Fine Tune Variable Resistance"
- board text removed: "Resistor & Parallel RC"

Commit message: Finished Tracing + DRC Check
Parts:
- removed RPONT: 0-100, DJ-FOOTPRINTS:RES-ADJ-TH_3P-L9.5-W9.5-P2.54-BR-BS
- added R22: 0-100, DJ-FOOTPRINTS:RES-ADJ-TH_3P-L9.5-W9.5-P2.54-BR-BS, F.Cu at (80.0, 96.0)
- moved R42 10.3 mm to (174.4, 61.6), turned to -90 degrees
- moved R43 7.63 mm to (177.8, 69.2), turned to 90 degrees
- moved R44 7.00 mm to (181.4, 61.6)
- moved R50 0.10 mm to (181.4, 91.6)
Routing:
- net Net-(J15-Pin_2): track 8.10 -> 87.9 mm
- net Net-(J7-Pin_2): track 0.00 -> 60.6 mm
- net Net-(J15-Pin_1): track 24.2 -> 59.5 mm
- net Net-(R49-Pad2): track 8.67 -> 39.1 mm
- net Net-(R46-Pad2): track 8.67 -> 33.3 mm
- net Net-(R43-Pad2): track 8.67 -> 31.8 mm
- net Net-(JP1-B): track 80.9 -> 58.3 mm
- net Net-(R47-Pad2): track 8.67 -> 23.9 mm
- net Net-(R48-Pad2): track 8.67 -> 23.6 mm
- net Net-(R41-Pad2): track 8.67 -> 23.1 mm
- net Net-(R44-Pad2): track 8.67 -> 22.3 mm
- net Net-(R45-Pad2): track 8.67 -> 19.9 mm
- net Net-(R40-Pad2): track 17.7 -> 27.6 mm
- net Net-(R42-Pad2): track 8.67 -> 17.9 mm
