File: RC-Substitution-Box.kicad_pcb (KiCad board)
At the start: 2 copper layers, 146.5 x 75.5 mm, 91 parts, among them J13 Screw_Terminal_01x02, J14 Screw_Terminal_01x02, J15 Screw_Terminal_01x02, J5 Screw_Terminal_01x02, J6 Screw_Terminal_01x02, J7 Screw_Terminal_01x02, SW2 208-12, SW3 208-12, SW4 208-12, SW5 208-12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

Commit message: Fix silkscreen labeling
-Values are too high
Other:
- board text added: "FIX SILKSCREEN LABELING"
